File: mm16.brd (EAGLE design)
At the start: 100 x 80 mm, 57 parts, among them IC101 ATMEGA32-PU, IC102 DS1337, IC103 MAX483CPA, IC201 LTV847, IC202 LTV847, IC203 LTV847, IC204 LTV847, Q1 32,768kHz

Commit message: Werte im Schema und Bohrungen im Layout hinzugefügt
Parts:
- C1, C101, C102, C103: value 10nF -> 100nF
- R201, R202, R203, R204, R205, R206, R207, R208, R209, R210, R211, R212, R213, R214, R215, R216: value (none) -> 220kΩ
Changed lines of the file:
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@@
 <element name="D207" library="diode" package="DO35-V" value="1N4148-V" x="39.37" y="62.23" rot="R270"/>
 <element name="D208" library="diode" package="DO35-V" value="1N4148-V" x="44.45" y="62.23" rot="R270"/>
-<element name="R201" library="passiv" package="0204V" value="" x="6.35" y="62.23" rot="R270"/>
-<element name="R202" library="passiv" package="0204V" value="" x="11.43" y="62.23" rot="R270"/>
-<element name="R203" library="passiv" package="0204V" value="" x="16.51" y="62.23" rot="R270"/>
-<element name="R204" library="passiv" package="0204V" value="" x="21.59" y="62.23" rot="R270"/>
-<element name="R205" library="passiv" package="0204V" value="" x="26.67" y="62.23" rot="R270"/>
-<element name="R206" library="passiv" package="0204V" value="" x="31.75" y="62.23" rot="R270"/>
-<element name="R207" library="passiv" package="0204V" value="" x="36.83" y="62.23" rot="R270"/>
-<element name="R208" library="passiv" package="0204V" value="" x="41.91" y="62.23" rot="R270"/>
+<element name="R201" library="passiv" package="0204V" value="220kΩ" x="6.35" y="62.23" rot="R270"/>
+<element name="R202" library="passiv" package="0204V" value="220kΩ" x="11.43" y="62.23" rot="R270"/>
+<element name="R203" library="passiv" package="0204V" value="220kΩ" x="16.51" y="62.23" rot="R270"/>
+<element name="R204" library="passiv" package="0204V" value="220kΩ" x="21.59" y="62.23" rot="R270"/>
+<element name="R205" library="passiv" package="0204V" value="220kΩ" x="26.67" y="62.23" rot="R270"/>
+<element name="R206" library="passiv" package="0204V" value="220kΩ" x="31.75" y="62.23" rot="R270"/>
+<element name="R207" library="passiv" package="0204V" value="220kΩ" x="36.83" y="62.23" rot="R270"/>
+<element name="R208" library="passiv" package="0204V" value="220kΩ" x="41.91" y="62.23" rot="R270"/>
 <element name="IC101" library="ic-mcu" package="DIL40" value="ATMEGA32-PU" x="46.99" y="31.75"/>
 <element name="IC203" library="ic-optokoppler" package="DIL16" value="LTV847" x="57.15" y="52.07" rot="R180"/>
@@
 <element name="D215" library="diode" package="DO35-V" value="1N4148-V" x="85.09" y="62.23" rot="R270"/>
 <element name="D216" library="diode" package="DO35-V" value="1N4148-V" x="90.17" y="62.23" rot="R270"/>
-<element name="R209" library="passiv" package="0204V" value="" x="52.07" y="62.23" rot="R270"/>
-<element name="R210" library="passiv" package="0204V" value="" x="57.15" y="62.23" rot="R270"/>
-<element name="R211" library="passiv" package="0204V" value="" x="62.23" y="62.23" rot="R270"/>
-<element name="R212" library="passiv" package="0204V" value="" x="67.31" y="62.23" rot="R270"/>
-<element name="R213" library="passiv" package="0204V" value="" x="72.39" y="62.23" rot="R270"/>
-<element name="R214" library="passiv" package="0204V" value="" x="77.47" y="62.23" rot="R270"/>
-<element name="R215" library="passiv" package="0204V" value="" x="82.55" y="62.23" rot="R270"/>
-<element name="R216" library="passiv" package="0204V" value="" x="87.63" y="62.23" rot="R270"/>
+<element name="R209" library="passiv" package="0204V" value="220kΩ" x="52.07" y="62.23" rot="R270"/>
+<element name="R210" library="passiv" package="0204V" value="220kΩ" x="57.15" y="62.23" rot="R270"/>
+<element name="R211" library="passiv" package="0204V" value="220kΩ" x="62.23" y="62.23" rot="R270"/>
+<element name="R212" library="passiv" package="0204V" value="220kΩ" x="67.31" y="62.23" rot="R270"/>
+<element name="R213" library="passiv" package="0204V" value="220kΩ" x="72.39" y="62.23" rot="R270"/>
+<element name="R214" library="passiv" package="0204V" value="220kΩ" x="77.47" y="62.23" rot="R270"/>
+<element name="R215" library="passiv" package="0204V" value="220kΩ" x="82.55" y="62.23" rot="R270"/>
+<element name="R216" library="passiv" package="0204V" value="220kΩ" x="87.63" y="62.23" rot="R270"/>
 <element name="SV101" library="stecker" package="ML6" value="" x="12.7" y="31.75" rot="R90"/>
 <element name="R101" library="passiv" package="0204V" value="10k" x="46.99" y="15.24"/>
@@
 <attribute name="OC_FARNELL" value="1007547" x="57.15" y="101.6" size="1.778" layer="27" rot="R180" display="off"/>
 </element>
-<element name="C101" library="passiv" package="C025-025X050" value="10nF" x="46.99" y="20.32"/>
-<element name="C102" library="passiv" package="C025-025X050" value="10nF" x="46.99" y="43.18" rot="R180"/>
-<element name="C103" library="passiv" package="C025-025X050" value="10nF" x="69.85" y="16.51" rot="R90"/>
+<element name="C101" library="passiv" package="C025-025X050" value="100nF" x="46.99" y="20.32"/>
+<element name="C102" library="passiv" package="C025-025X050" value="100nF" x="46.99" y="43.18" rot="R180"/>
+<element name="C103" library="passiv" package="C025-025X050" value="100nF" x="69.85" y="16.51" rot="R90"/>
 <element name="IC102" library="ic-controller" package="DIL08" value="DS1337" x="21.59" y="16.51"/>
 <element name="Q1" library="passiv" package="TC38H" value="32,768kHz" x="17.78" y="8.89" rot="R270"/>
-<element name="C1" library="passiv" package="C025-025X050" value="10nF" x="29.21" y="16.51" rot="R270"/>
+<element name="C1" library="passiv" package="C025-025X050" value="100nF" x="29.21" y="16.51" rot="R270"/>
 <element name="X2" library="anschluss" package="WAGO_236-408" value="" x="26.67" y="71.12" rot="R180"/>
 <element name="X3" library="anschluss" package="WAGO_236-408" value="" x="72.39" y="71.12" rot="R180"/>
