File: mm16.sch (EAGLE design)
At the start: 58 parts, among them IC101 ATMEGA32-PU, IC102 DS1337, IC103 MAX483CPA, IC201 LTV847, IC202 LTV847, IC203 LTV847, IC204 LTV847, Q1 32,768kHz

Commit message: Batteriehalter ausgetauscht
Parts:
- G1: value CR2032V -> KZH20PCB-V; device battery:CR2032V -> batterie:KZH20PCB-V
Connections:
- net N$21: no longer G1.+@1
Other:
- moved on the sheet: G1
Changed lines of the file:
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@@
 <part name="D1" library="diode" deviceset="1N4148" device="-7"/>
 <part name="D2" library="diode" deviceset="1N4148" device="-7"/>
-<part name="G1" library="battery" deviceset="CR2032V" device=""/>
 <part name="GND39" library="versorgung" deviceset="GND" device=""/>
 <part name="S1" library="switch-dil" deviceset="P103" device=""/>
@@
 <part name="X3" library="anschluss" deviceset="WAGO_236-408" device=""/>
 <part name="R1" library="passiv" deviceset="R_" device="0204/2V" value="120Ω"/>
+<part name="G1" library="batterie" deviceset="KZH20" device="PCB-V"/>
 </parts>
 <sheets>
@@
 <instance part="D1" gate="G$1" x="170.18" y="157.48"/>
 <instance part="D2" gate="G$1" x="205.74" y="157.48" rot="R180"/>
-<instance part="G1" gate="1" x="218.44" y="152.4" rot="R90"/>
-<instance part="GND39" gate="1" x="218.44" y="144.78"/>
+<instance part="GND39" gate="1" x="218.44" y="142.24"/>
 <instance part="S1" gate="1" x="132.08" y="116.84" rot="R90"/>
 <instance part="P+2" gate="1" x="83.82" y="167.64"/>
@@
 <instance part="X6" gate=".2" x="165.1" y="22.86" rot="R180"/>
 <instance part="R1" gate="G$1" x="157.48" y="15.24" rot="R90"/>
+<instance part="G1" gate="1" x="218.44" y="149.86"/>
 </instances>
 <busses>
@@
 </segment>
 <segment>
-<pinref part="G1" gate="1" pin="-"/>
-<pinref part="GND39" gate="1" pin="GND"/>
-</segment>
-<segment>
 <pinref part="S1" gate="1" pin="C"/>
 <pinref part="GND44" gate="1" pin="GND"/>
 <wire x1="139.7" y1="116.84" x2="142.24" y2="116.84" width="0.1524" layer="91"/>
 <wire x1="142.24" y1="116.84" x2="142.24" y2="114.3" width="0.1524" layer="91"/>
+</segment>
+<segment>
+<pinref part="GND39" gate="1" pin="GND"/>
+<pinref part="G1" gate="1" pin="-"/>
+<wire x1="218.44" y1="144.78" x2="218.44" y2="147.32" width="0.1524" layer="91"/>
 </segment>
 </net>
@@
 <segment>
 <pinref part="D2" gate="G$1" pin="A"/>
+<wire x1="208.28" y1="157.48" x2="218.44" y2="157.48" width="0.1524" layer="91"/>
+<wire x1="218.44" y1="157.48" x2="218.44" y2="154.94" width="0.1524" layer="91"/>
 <pinref part="G1" gate="1" pin="+"/>
-<wire x1="208.28" y1="157.48" x2="218.44" y2="157.48" width="0.1524" layer="91"/>
-<pinref part="G1" gate="1" pin="+@1"/>
-<wire x1="218.44" y1="157.48" x2="218.44" y2="154.94" width="0.1524" layer="91"/>
 </segment>
 </net>
@@
 </sheet>
 </sheets>
-<errors>
-</errors>
 </schematic>
 </drawing>
