File: out8.brd (EAGLE design)
At the start: 100 x 80 mm, 38 parts, among them IC1 74HC595N, K301 S202S02, K302 S202S02, K303 S202S02, K304 S202S02, K305 S202S02, K306 S202S02, K307 S202S02, K308 S202S02

Commit message: Boards beschriftet
Parts:
- C101: value 10nF -> 100nF
- F1, F2, F3, F4, F5, F6, F7, F8: value (none) -> 2T
- R301, R302, R303, R304, R305, R306, R307, R308: value (none) -> 180Ω
Other:
- board text added: "STR 7/12"
- board text added: "out8 Rev.1"
