File: dig_ac230.brd (EAGLE design)
At the start: 100 x 85 mm, 142 parts, among them IC201 ATMEGA32A-AU, IC202 DS1337S, IC203 MAX487CSA, IC204 74HC166D, IC301 LTV-356T, IC302 LTV-356T, IC303 LTV-356T, IC304 LTV-356T, IC305 LTV-356T, IC306 LTV-356T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

Commit message: Batteriespannungsdioden versetzt
Parts:
- moved D103 37.6 mm to (21.6, 24.1), flipped to the bottom, turned to 0 degrees
- moved D102 36.2 mm to (21.6, 26.7), flipped to the bottom
Routing:
- net N$64: track 58.6 -> 14.2 mm, vias 4 -> 1
- net N$21: track 38.0 -> 76.9 mm, vias 1 -> 2
- net +5V: track 312.0 -> 316.4 mm
