File: hardware/dmi.brd (EAGLE design)
At the start: 76.5 x 50.8 mm, 53 parts, among them IC1 ATMEGA328-A, IC2 MAX487CSA, IC3 78SO05, IC4 LTV-354T, IC5 LTV-356T, Q1 BC337, Q2 BC337, X1 AKL_183-02, X2 AKL_183-02, X3 AKL_183-02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

Commit message: Türinnenmodul überarbeitet
Parts:
- IC1: value ATMEGA328-A -> ATMEGA328PB-AU
- moved C1 0.63 mm to (48.3, 27.9), turned to 270 degrees
Connections:
- net +5V: no longer IC1.6
- net GND: no longer IC1.3
Routing:
- net GND: track 106.3 -> 103.0 mm
- net +5V: track 149.1 -> 145.9 mm
